File: schematics/65C02_Computer_DEC-2/65C02_Computer.sch (KiCad schematic (older format))
At the start: 29 parts, among them J1 CLK Jumper, J2 Expansion port, SW1 RESET, U1 74HC14, U2 28C256, U3 65C02S, U4 74HC00, U5 62256, X1 1MHz

Commit message: Updating new schematic for BW-DEC-2
Parts:
- removed U4: 74HC00, Package_DIP:DIP-14_W7.62mm_Socket, symbol 74xx:74HC00
- removed U?: CD74AC138, Package_DIP:DIP-16_W7.62mm, symbol 74xx_IEEE:CD74AC138
- added R4: 3K3, Resistor_THT:R_Axial_DIN0207_L6.3mm_D2.5mm_P7.62mm_Horizontal, symbol Device:R
- added U7: CD74AC138, Package_DIP:DIP-16_W7.62mm, symbol 65C02_Computer-rescue:CD74AC138-65C02_Computer-cache
- added U? (x2): SN74HC11, Package_DIP:DIP-14_W7.62mm, symbol 74xx:SN74HC11
- U6: renamed from U?; symbol Logic_Programmable:BW-DEC-2 -> 65C02_Computer-rescue:BW-DEC-2-Logic_Programmable
- renumbered C4 to C10, C5 to C4, C6 to C5, C7 to C6, C8 to C7, C9 to C8, C10 to C9, R4 to R5, R5 to R6, R6 to R7
Connections:
- net labels added: ~AIRQ, ~V1IRQ, ~V2IRQ
- wire segments 257 -> 265
- no-connect marks 19 -> 18
Changed lines of the file:
@@
 CLK
-$Comp
-L 74xx:74HC00 U4
-U 1 1 5E16D50B
-P 3600 6300
-F 0 "U4" H 3600 6625 50  0000 C CNN
-F 1 "74HC00" H 3600 6534 50  0000 C CNN
-F 2 "Package_DIP:DIP-14_W7.62mm_Socket" H 3600 6300 50  0001 C CNN
-F 3 "http://www.ti.com/lit/gpn/sn74hc00" H 3600 6300 50  0001 C CNN
-	1    3600 6300
-	1    0    0    -1
-$EndComp
 $Comp
 L Oscillator:ACO-xxxMHz X1
@@
 R~W
 $Comp
-L Device:R R5
+L Device:R R6
 U 1 1 5E1F5B26
 P 8050 5450
-F 0 "R5" V 7950 5450 50  0000 C CNN
+F 0 "R6" V 7950 5450 50  0000 C CNN
 F 1 "20K" V 8050 5450 50  0000 C CNN
 F 2 "Resistor_THT:R_Axial_DIN0207_L6.3mm_D2.5mm_P7.62mm_Horizontal" V 7980 5450 50  0001 C CNN
@@
 $EndComp
 $Comp
-L Device:CP C4
+L Device:CP C10
 U 1 1 5E2337BD
 P 8350 5050
-F 0 "C4" H 8468 5096 50  0000 L CNN
+F 0 "C10" H 8468 5096 50  0000 L CNN
 F 1 "1uF" H 8468 5005 50  0000 L CNN
 F 2 "Capacitor_THT:CP_Radial_D5.0mm_P2.50mm" H 8388 4900 50  0001 C CNN
@@
 $EndComp
 $Comp
-L Device:R R4
+L Device:R R5
 U 1 1 5E3A85D8
 P 7750 5150
-F 0 "R4" V 7650 5150 50  0000 C CNN
+F 0 "R5" V 7650 5150 50  0000 C CNN
 F 1 "20K" V 7750 5150 50  0000 C CNN
 F 2 "Resistor_THT:R_Axial_DIN0207_L6.3mm_D2.5mm_P7.62mm_Horizontal" V 7680 5150 50  0001 C CNN
@@
 ~RES
 $Comp
-L Device:R R6
+L Device:R R7
 U 1 1 5E552FBE
 P 8700 5450
-F 0 "R6" V 8600 5450 50  0000 C CNN
+F 0 "R7" V 8600 5450 50  0000 C CNN
 F 1 "51K" V 8700 5450 50  0000 C CNN
 F 2 "Resistor_THT:R_Axial_DIN0207_L6.3mm_D2.5mm_P7.62mm_Horizontal" V 8630 5450 50  0001 C CNN
@@
 $EndComp
 $Comp
-L Device:C C10
+L Device:C C9
 U 1 1 5E3E14F5
 P 8300 3600
-F 0 "C10" H 8415 3646 50  0000 L CNN
+F 0 "C9" H 8415 3646 50  0000 L CNN
 F 1 "0.1uF" H 8415 3555 50  0000 L CNN
 F 2 "Capacitor_THT:C_Disc_D3.4mm_W2.1mm_P2.50mm" H 8338 3450 50  0001 C CNN
@@
 $EndComp
 $Comp
-L Device:C C9
+L Device:C C8
 U 1 1 5E3E1910
 P 7850 3600
-F 0 "C9" H 7965 3646 50  0000 L CNN
+F 0 "C8" H 7965 3646 50  0000 L CNN
 F 1 "0.1uF" H 7965 3555 50  0000 L CNN
 F 2 "Capacitor_THT:C_Disc_D3.4mm_W2.1mm_P2.50mm" H 7888 3450 50  0001 C CNN
@@
 $EndComp
 $Comp
-L Device:C C8
+L Device:C C7
 U 1 1 5E3E1BD5
 P 7400 3600
-F 0 "C8" H 7515 3646 50  0000 L CNN
+F 0 "C7" H 7515 3646 50  0000 L CNN
 F 1 "0.1uF" H 7515 3555 50  0000 L CNN
 F 2 "Capacitor_THT:C_Disc_D3.4mm_W2.1mm_P2.50mm" H 7438 3450 50  0001 C CNN
@@
 $EndComp
 $Comp
-L Device:C C6
+L Device:C C5
 U 1 1 5E3E2103
 P 6500 3600
-F 0 "C6" H 6615 3646 50  0000 L CNN
+F 0 "C5" H 6615 3646 50  0000 L CNN
 F 1 "0.1uF" H 6615 3555 50  0000 L CNN
 F 2 "Capacitor_THT:C_Disc_D3.4mm_W2.1mm_P2.50mm" H 6538 3450 50  0001 C CNN
@@
 $EndComp
 $Comp
-L Device:C C5
+L Device:C C4
 U 1 1 5E3E2489
 P 6050 3600
-F 0 "C5" H 6165 3646 50  0000 L CNN
+F 0 "C4" H 6165 3646 50  0000 L CNN
 F 1 "0.1uF" H 6165 3555 50  0000 L CNN
 F 2 "Capacitor_THT:C_Disc_D3.4mm_W2.1mm_P2.50mm" H 6088 3450 50  0001 C CNN
@@
 Text GLabel 2700 2600 2    50   Input ~ 0
 d[0..7]
-$Comp
-L 74xx:74HC00 U4
-U 5 1 5E5C6EF1
-P 2050 6850
-F 0 "U4" H 2280 6896 50  0000 L CNN
-F 1 "74HC00" H 2280 6805 50  0000 L CNN
-F 2 "Package_DIP:DIP-14_W7.62mm_Socket" H 2050 6850 50  0001 C CNN
-F 3 "http://www.ti.com/lit/gpn/sn74hc00" H 2050 6850 50  0001 C CNN
-	5    2050 6850
-	1    0    0    -1
-$EndComp
-Text GLabel 2050 6250 1    50   Input ~ 0
+Text GLabel 2050 6350 1    50   Input ~ 0
 +5V
-Text GLabel 2050 7450 3    50   Input ~ 0
+Text GLabel 2050 7350 3    50   Input ~ 0
 GND
 Text GLabel 4100 2850 0    50   Input ~ 0
@@
 Text GLabel 1250 7350 3    50   Input ~ 0
 GND
-Text GLabel 3300 6400 0    50   Input ~ 0
-+5V
-Text GLabel 3300 6200 0    50   Input ~ 0
-+5V
-NoConn ~ 3900 6300
 Text GLabel 7700 1750 2    50   Output ~ 0
 ~RAM_CS
@@
 $EndComp
 $Comp
-L Device:C C7
+L Device:C C6
 U 1 1 5E3E1DA8
 P 6950 3600
-F 0 "C7" H 7065 3646 50  0000 L CNN
+F 0 "C6" H 7065 3646 50  0000 L CNN
 F 1 "0.1uF" H 7065 3555 50  0000 L CNN
 F 2 "Capacitor_THT:C_Disc_D3.4mm_W2.1mm_P2.50mm" H 6988 3450 50  0001 C CNN
@@
 $EndComp
 $Comp
-L Logic_Programmable:BW-DEC-2 U?
+L 65C02_Computer-rescue:BW-DEC-2-Logic_Programmable U6
 U 1 1 609E77AF
 P 6850 2000
-F 0 "U?" H 6850 2981 50  0000 C CNN
+F 0 "U6" H 6850 2981 50  0000 C CNN
 F 1 "BW-DEC-2" H 6850 2890 50  0000 C CNN
 F 2 "Package_DIP:DIP-24_W7.62mm" H 6850 1950 50  0001 C CNN
@@
 	2700 2600 2600 2600
 Wire Wire Line
-	2050 6250 2050 6350
-Wire Wire Line
-	2050 7350 2050 7450
-Wire Wire Line
 	4100 2850 4200 2850
 Wire Wire Line
@@
 Wire Wire Line
 	8350 1450 8450 1450
-$Comp
-L 74xx_IEEE:CD74AC138 U?
-U 1 1 60D0F4F3
-P 9000 1650
-F 0 "U?" H 9000 2281 50  0000 C CNN
-F 1 "CD74AC138" H 9000 2190 50  0000 C CNN
-F 2 "Package_DIP:DIP-16_W7.62mm" H 9000 1650 50  0001 C CNN
-F 3 "" H 9000 1650 50  0001 C CNN
-	1    9000 1650
-	1    0    0    -1
-$EndComp
 NoConn ~ 9550 2150
 NoConn ~ 9550 2050
@@
 Wire Wire Line
 	6250 1550 6250 1600
+Text GLabel 8500 1250 0    50   Input ~ 0
++5V
+Wire Wire Line
+	8500 1250 9000 1250
+Wire Wire Line
+	9000 2350 9000 2400
+$Comp
+L 65C02_Computer-rescue:CD74AC138-65C02_Computer-cache U7
+U 1 1 60AC9AD5
+P 9000 1650
+F 0 "U7" H 9000 2231 50  0000 C CNN
+F 1 "CD74AC138" H 9000 2140 50  0000 C CNN
+F 2 "Package_DIP:DIP-16_W7.62mm" H 9000 1650 50  0001 C CNN
+F 3 "" H 9000 1650 50  0001 C CNN
+	1    9000 1650
+	1    0    0    -1
+$EndComp
+Text GLabel 3700 1600 0    50   Input ~ 0
+~AIRQ
+Text GLabel 3700 1800 0    50   Input ~ 0
+~V1IRQ
+Text GLabel 3700 2000 0    50   Input ~ 0
+~V2IRQ
+Wire Wire Line
+	3700 1600 4050 1600
+Wire Wire Line
+	4050 1600 4050 1700
+Wire Wire Line
+	3700 1800 4050 1800
+Wire Wire Line
+	3700 2000 4050 2000
+Wire Wire Line
+	4050 2000 4050 1900
+$Comp
+L Device:R R4
+U 1 1 60B10BDF
+P 4050 1300
+F 0 "R4" V 3950 1300 50  0000 C CNN
+F 1 "3K3" V 4050 1300 50  0000 C CNN
+F 2 "Resistor_THT:R_Axial_DIN0207_L6.3mm_D2.5mm_P7.62mm_Horizontal" V 3980 1300 50  0001 C CNN
+F 3 "~" H 4050 1300 50  0001 C CNN
+	1    4050 1300
+	-1   0    0    1
+$EndComp
+Wire Wire Line
+	4050 1450 4050 1600
+Connection ~ 4050 1600
+Text GLabel 4050 1000 1    50   Input ~ 0
++5V
+Wire Wire Line
+	4050 1150 4050 1000
+Text GLabel 4900 1800 2    50   Output ~ 0
+~IRQ
+Wire Wire Line
+	4650 1800 4900 1800
+$Comp
+L 74xx:SN74HC11 U?
+U 2 1 609D7628
+P 4350 1800
+F 0 "U?" H 4350 2125 50  0000 C CNN
+F 1 "SN74HC11" H 4350 2034 50  0000 C CNN
+F 2 "Package_DIP:DIP-14_W7.62mm" H 4350 1800 50  0001 C CNN
+F 3 "https://www.ti.com/lit/ds/symlink/sn54hc11-sp.pdf" H 4350 1800 50  0001 C CNN
+	2    4350 1800
+	1    0    0    -1
+$EndComp
+$Comp
+L 74xx:SN74HC11 U?
+U 4 1 609D9475
+P 2050 6850
+F 0 "U?" H 2280 6896 50  0000 L CNN
+F 1 "SN74HC11" H 2280 6805 50  0000 L CNN
+F 2 "Package_DIP:DIP-14_W7.62mm" H 2050 6850 50  0001 C CNN
+F 3 "https://www.ti.com/lit/ds/symlink/sn54hc11-sp.pdf" H 2050 6850 50  0001 C CNN
+	4    2050 6850
+	1    0    0    -1
+$EndComp
 Wire Bus Line
 	3100 5450 3100 5650

Commit message: schematics for computer with BW-DEC-2
Parts:
- removed U? (x2): SN74HC11, Package_DIP:DIP-14_W7.62mm, symbol 74xx:SN74HC11
- added C11, C12: 0.1uF, Capacitor_THT:C_Disc_D3.4mm_W2.1mm_P2.50mm, symbol Device:C
- added U4: SN74HC11, Package_DIP:DIP-14_W7.62mm, symbol 65C02_Computer-rescue:SN74HC11-65C02_Computer-cache
- U1: footprint Package_DIP:DIP-14_W7.62mm_Socket -> Package_DIP:DIP-14_W7.62mm
- U6: footprint Package_DIP:DIP-24_W7.62mm -> Package_DIP:DIP-24_W7.62mm_Socket
- renumbered C11 to C13, C12 to C14
Connections:
- net ~IRQX is gone; now on net ~IRQ_OD: J2.26 (Pin_26)
- net ~ROM_OE is gone; now on net ~OE: U2.22 (~OE)
- net +5V: now also U6.24 (VCC), C11.1, C12.1, U4.1, U4.10, U4.11, U4.13, U4.14 (VCC), U4.2, U4.9
- net GND: now also C11.2, C12.2, U4.7 (GND)
- net R~W: no longer U5.27 (~WE)
- net ~IRQ: now also U4.6
- net ~OE: now also U5.22 (~OE)
- net ~RAM_CS: no longer U5.22 (~OE)
- net ~V1IRQ: now also U4.4
- net ~V2IRQ: now also U4.5
- net ~WE: now also U5.27 (~WE)
- net ~AIRQ renamed ~IRQ_OD
- net ~IRQ_OD: now also U4.3
- no-connect marks 18 -> 19
Other:
- moved on the sheet: C13, C14, U1B, U1C
